File: Hardware/Bus_switch.kicad_sch (KiCad schematic)
At the start: 15 parts, among them J3 Conn_01x04_Pin, U1 SN74CB3Q3384APW

Commit message: idea schematic
Other:
- company: (none) -> MiniModucard System
- title: MMS3 Hat template small (Change Me) -> MMS3 Hat Meter/Source
Changed lines of the file:
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@@
 	(paper "A4")
 	(title_block
-		(title "MMS3 Hat template small (Change Me)")
-		(date "2026-02-25")
+		(title "MMS3 Hat Meter/Source")
+		(date "2026-06-24")
 		(rev "A")
-		(comment 1 "Made by Wojciech Szafrański")
+		(company "MiniModucard System")
+		(comment 1 "Wojciech Szafrański")
 		(comment 2 "Designed in poland")
 	)
