File: Hardware/Bus_switch.kicad_sch (KiCad schematic)
At the start: 15 parts, among them J3 Conn_01x04_Pin, U1 SN74CB3Q3384APW

Commit message: all to 0603
Parts:
- removed R1: 330Ω, PCM_JLCPCB:R_0402, symbol PCM_JLCPCB-Resistors:0402,330Ω
- removed R10, R11, R2, R3, R4, R5, R6, R7, R8, R9: 10kΩ, PCM_JLCPCB:R_0402, symbol PCM_JLCPCB-Resistors:0402,10kΩ
- added R1: 1kΩ, PCM_JLCPCB:R_0603, symbol PCM_JLCPCB-Resistors:0603,1kΩ
- added R10, R4, R6: 10kΩ, PCM_JLCPCB:R_0603, symbol PCM_JLCPCB-Resistors:0603,10kΩ
Connections:
- net +3V3: now also R10.2, R4.2, R6.2
- net Chainbus.SCL: now also R6.1
- net Chainbus.SDA: now also R10.1
- net SEL1: now also R1.1, R4.1
- net at D3.1: now also R1.2
