File: Hardware/ID_EEPROM.kicad_sch (KiCad schematic)
At the start: 2 parts, among them U2 M24C64

Commit message: idea schematic
Other:
- company: (none) -> MiniModucard System
- title: MMS3 Hat template small (Change Me) -> MMS3 Hat Meter/Source
Changed lines of the file:
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@@
 	(paper "A4")
 	(title_block
-		(title "MMS3 Hat template small (Change Me)")
-		(date "2026-02-25")
+		(title "MMS3 Hat Meter/Source")
+		(date "2026-06-24")
 		(rev "A")
-		(comment 1 "Made by Wojciech Szafrański")
+		(company "MiniModucard System")
+		(comment 1 "Wojciech Szafrański")
 		(comment 2 "Designed in poland")
 	)
