File: Hardware/Interboard_connector.kicad_sch (KiCad schematic)
At the start: 2 parts, among them J1 Chainbus in, J2 Chainbus Out

Commit message: fixed reserved pins
Connections:
- net R1: now reaches J2.25 (Pin_25)
- net R1: now also J1.25 (Pin_25)
- net R2: now reaches J2.27 (Pin_27)
- net R2: now also J1.27 (Pin_27)
- no-connect marks 5 -> 1
Changed lines of the file:
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@@
-	)
-	(no_connect
-		(at 113.03 53.34)
-	)
-	(no_connect
-		(at 115.57 53.34)
 	)
 	(no_connect
 		(at 176.53 66.04)
-	)
-	(no_connect
-		(at 191.77 53.34)
-	)
-	(no_connect
-		(at 189.23 53.34)
 	)
 	(bus_entry
@@
 		)
 	)
+	(label "R2"
+		(at 191.77 53.34 0)
+		(effects
+			(font
+				(size 1.27 1.27)
+			)
+			(justify left bottom)
+		)
+	)
 	(label "Chainbus.MOSI"
 		(at 113.03 67.31 270)
@@
 		)
 	)
+	(label "R1"
+		(at 189.23 53.34 0)
+		(effects
+			(font
+				(size 1.27 1.27)
+			)
+			(justify left bottom)
+		)
+	)
 	(label "SEL4"
 		(at 163.83 76.2 270)
@@
 		)
 	)
+	(label "R2"
+		(at 115.57 53.34 0)
+		(effects
+			(font
+				(size 1.27 1.27)
+			)
+			(justify left bottom)
+		)
+	)
 	(label "Chainbus.SDA"
 		(at 179.07 67.31 270)
@@
 		)
 	)
+	(label "R1"
+		(at 113.03 53.34 0)
+		(effects
+			(font
+				(size 1.27 1.27)
+			)
+			(justify left bottom)
+		)
+	)
