File: Hardware/MMS3_hat_templates.kicad_sch (KiCad schematic)
At the start: 12 parts, among them U4 AMS1117

Commit message: idea schematic
Parts:
- added C4: C, symbol Device:C
- added C7, C8: 100nF, PCM_JLCPCB:C_0603, symbol PCM_JLCPCB-Capacitors:0603,100nF
- added D2: D_Zener, symbol Device:D_Zener
- added J6: Conn_01x02, symbol Connector_Generic:Conn_01x02
- added Q1, Q9: PMOS, symbol Simulation_SPICE:PMOS
- added Q10, Q2, Q3, Q4, Q5, Q6, Q7, Q8: NMOS, symbol Simulation_SPICE:NMOS
- added R14: shunt, symbol Device:R
- added R15, R16, R25, R28: 0Ω, PCM_JLCPCB:R_0603, symbol PCM_JLCPCB-Resistors:0603,0Ω
- added R17, R18, R19, R20, R21, R22, R23, R24, R26, R27, R29, R30, R31, R32, R33: R, symbol Device:R
- added U3, U6: LM358DR2G, PCM_JLCPCB:SOIC-8_L5.0-W4.0-P1.27-LS6.0-BL, symbol PCM_JLCPCB-Analog:Op-Amp, LM358DR2G
Connections:
- net GND: now also C4.2, C7.2, C8.2, D2.2 (A), R14.2, R17.2, R22.1, R24.1, R26.1, R27.1, R31.1, R33.2, U3.4 (GND), U3.5 (2IN+), U3.6 (2IN-), U6.4 (GND)
- net VIN_CHAINBUS: now also C7.1, C8.1, Q1.3 (S), U3.8 (VCC), U6.8 (VCC)
- new net: Q5.1 (D), Q6.1 (D), Q7.1 (D), R22.2, R23.1, U3.2 (1IN-)
- new net: Q7.3 (S), R27.2
- new net: Q10.1 (D), R28.2
- new net: R25.1, R28.1, U6.6 (2IN-)
- new net: Q8.1 (D), R25.2
- new net: Q1.2 (G), R16.2
- new net: Q4.3 (S), R21.1
- new net: R14.1, R15.2
- new net: Q3.3 (S), R20.1
- new net: Q5.3 (S), R26.2
- new net: C4.1, R29.2, U6.5 (2IN+)
- new net: Q2.3 (S), R19.1
- new net: Q6.3 (S), R24.2
- new net: Q8.3 (S), R30.2
- new net Amm_ADC: R23.2, U3.1 (1OUT)
- new net Amp_+: J6.2 (Pin_2), Q9.1 (D), R15.1, U3.3 (1IN+), U6.3 (1IN+)
- new net OP_Gate_-: R32.2, R33.1, U6.2 (1IN-)
- new net OP_Gate_Out: Q10.3 (S), R32.1, U6.1 (1OUT)
- new net PWM: R29.1
- new net Pmos_Gate: R16.1, U6.7 (2OUT)
- new net Volt_+: J6.1 (Pin_1), Q1.1 (D), Q2.1 (D), Q3.1 (D), Q4.1 (D), Q9.3 (S), R18.1, R30.1, R31.2
- new net Volt_ADC: D2.1 (K), R17.1, R18.2, R19.2, R20.2, R21.2
- no-connect marks 0 -> 9
Other:
- added sheet CH32V003 (CH32V003.kicad_sch)
- note added: "Ammeter"
- note added: "MCU CH32V003"
- note added: "Output Connector"
- note added: "Output Gate Driver"
- note added: "Voltmeter"
- note removed: "<-- Use those connections"
- title: MMS3 Hat template small (Change Me) -> MMS3 Hat Meter/Source
- moved on the sheet: C16, C18, H1, H2, H3, H4, H5, H6, H7, H8, H9, U4
