File: Hardware/CH32V003.kicad_sch (KiCad schematic)
At the start: 10 parts, among them J7 Program, U5 CH32V003FxPx, X2 X322525MOB4SI

Commit message: all to 0603
Parts:
- removed R12: 10kΩ, PCM_JLCPCB:R_0402, symbol PCM_JLCPCB-Resistors:0402,10kΩ
- removed R13: 330Ω, PCM_JLCPCB:R_0402, symbol PCM_JLCPCB-Resistors:0402,330Ω
- added R12: 10kΩ, PCM_JLCPCB:R_0603, symbol PCM_JLCPCB-Resistors:0603,10kΩ
- added R13: 1kΩ, PCM_JLCPCB:R_0603, symbol PCM_JLCPCB-Resistors:0603,1kΩ
- C3, C5, D5, S1, X2: now not fitted; now left out of the parts list
Connections:
- net +3V3: now also R12.1
- net PD6 (RX): now also R13.1
- net PD7 (NRST): now also R12.2
- net at D5.2: now also R13.2

Commit message: final touches, readme
Changed lines of the file:
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@@
 	)
 	(label "CH32V003.SCL"
-		(at 58.42 93.98 0)
+		(at 58.42 97.79 0)
 		(effects
 			(font
@@
 	)
 	(label "CH32V003.SDA"
-		(at 58.42 97.79 0)
+		(at 58.42 93.98 0)
 		(effects
 			(font
