File: Hardware/MMS3_hat_Meter-Source.kicad_sch (KiCad schematic)
At the start: 87 parts, among them J6 Conn_01x02, Q12 2N7002, Q13 2N7002, Q14 2N7002, Q15 2N7002, Q18 2N7002, Q19 2N7002, Q20 2N7002, Q3 S60N04F, Q4 AGM40P25A, U3 LM358DR2G, U4 AMS1117, U6 LM358DR2G, U7 LM358DR2G

Commit message: back to m2.5
Parts:
- H1: value M3 Mount -> M2.5 mount; footprint MountingHole:MountingHole_3.2mm_M3_DIN965_Pad_TopOnly -> MountingHole:MountingHole_2.7mm_M2.5_DIN965_Pad_TopOnly
- H2, H3, H4: value M3 mount -> M2.5 mount; footprint MountingHole:MountingHole_3.2mm_M3_DIN965 -> MountingHole:MountingHole_2.7mm_M2.5
Changed lines of the file:
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@@
 			)
 		)
-		(property "Value" "M3 mount"
+		(property "Value" "M2.5 mount"
 			(at 114.3 384.8099 0)
 			(show_name no)
@@
 			)
 		)
-		(property "Footprint" "MountingHole:MountingHole_3.2mm_M3_DIN965"
+		(property "Footprint" "MountingHole:MountingHole_2.7mm_M2.5"
 			(at 111.76 383.54 0)
 			(hide yes)
@@
 			)
 		)
-		(property "Value" "M3 mount"
+		(property "Value" "M2.5 mount"
 			(at 114.3 389.8899 0)
 			(show_name no)
@@
 			)
 		)
-		(property "Footprint" "MountingHole:MountingHole_3.2mm_M3_DIN965"
+		(property "Footprint" "MountingHole:MountingHole_2.7mm_M2.5"
 			(at 111.76 388.62 0)
 			(hide yes)
@@
 			)
 		)
-		(property "Value" "M3 mount"
+		(property "Value" "M2.5 mount"
 			(at 114.3 394.9699 0)
 			(show_name no)
@@
 			)
 		)
-		(property "Footprint" "MountingHole:MountingHole_3.2mm_M3_DIN965"
+		(property "Footprint" "MountingHole:MountingHole_2.7mm_M2.5"
 			(at 111.76 393.7 0)
 			(hide yes)
@@
 			)
 		)
-		(property "Value" "M3 Mount"
+		(property "Value" "M2.5 mount"
 			(at 97.79 384.8099 0)
 			(show_name no)
@@
 			)
 		)
-		(property "Footprint" "MountingHole:MountingHole_3.2mm_M3_DIN965_Pad_TopOnly"
+		(property "Footprint" "MountingHole:MountingHole_2.7mm_M2.5_DIN965_Pad_TopOnly"
 			(at 95.25 384.81 0)
 			(hide yes)

Commit message: final touches, readme
Parts:
- removed R25, R28, R55: 0Ω, PCM_JLCPCB:R_0603, symbol PCM_JLCPCB-Resistors:0603,0Ω
- added J10, J11, J9: Conn_01x02, Connector_PinHeader_2.54mm:PinHeader_1x02_P2.54mm_Vertical, symbol Connector_Generic:Conn_01x02
- added J8: Conn_01x02, Connector_JST:JST_XH_B2B-XH-A_1x02_P2.50mm_Vertical, symbol Connector_Generic:Conn_01x02
Connections:
- net Free: now also J8.1 (Pin_1)
- net GND: now also R53.2, J8.2 (Pin_2); no longer R53.1
- net Mosfet_Feedback: now also J10.1 (Pin_1), J11.1 (Pin_1), J9.1 (Pin_1)
- net OP_Gate_-: now also R31.1, R53.1; no longer R31.2, R53.2
- net OP_Gate_Out: now also R31.2; no longer R31.1
- net at Q18.3 (D): now also J9.2 (Pin_2)
- net at Q20.3 (D): now also J11.2 (Pin_2)
- net at Q19.3 (D): now also J10.2 (Pin_2)
Other:
- note added: "Output Gate Driver - NMOS"
- note added: "Output Gate Driver - PMOS"
- note removed: "Output Gate Driver"
