File: Hardware/MMS3_hat_Meter-Source.kicad_pcb (KiCad board)
At the start: 2 copper layers, 100 x 50 mm, 107 parts, among them J1 Chainbus in, J2 Chainbus Out, J3 Conn_01x04_Pin, J4 AMASS XT60 Male, J5 AMASS XT60 Female, J6 Conn_01x02, J7 Program, Q12 2N7002, Q13 2N7002, Q14 2N7002, Q15 2N7002, Q18 2N7002, Q19 2N7002, Q20 2N7002, Q3 S60N04F, Q4 AGM40P25A, U1 SN74CB3Q3384APW, U2 M24C64, U3 LM358DR2G, U4 AMS1117, U5 CH32V003FxPx, U6 LM358DR2G, U7 LM358DR2G

Commit message: back to m2.5
Parts:
- H1: value M3 Mount -> M2.5 mount; footprint MountingHole:MountingHole_3.2mm_M3_DIN965_Pad_TopOnly -> MountingHole:MountingHole_2.7mm_M2.5_DIN965_Pad_TopOnly
- H2, H3: value M3 mount -> M2.5 mount; footprint MountingHole:MountingHole_3.2mm_M3_DIN965 -> MountingHole:MountingHole_2.7mm_M2.5
- H4: value M3 mount -> M2.5 mount
Changed lines of the file:
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@@
 		)
 	)
-	(footprint "MountingHole:MountingHole_3.2mm_M3_DIN965_Pad_TopOnly"
+	(footprint "MountingHole:MountingHole_2.7mm_M2.5_DIN965_Pad_TopOnly"
 		(layer "F.Cu")
 		(at 82 92)
-		(descr "Mounting Hole 3.2mm, M3, generated by kicad-footprint-generator mountinghole.py")
-		(tags "mountinghole M3 DIN965")
+		(descr "Mounting Hole 2.7mm, M2.5, generated by kicad-footprint-generator mountinghole.py")
+		(tags "mountinghole M2.5 DIN965")
 		(property "Reference" "H1"
-			(at 0 -3.75 0)
+			(at 0 -3.3 0)
 			(layer "F.SilkS")
 			(effects
@@
 			)
 		)
-		(property "Value" "M3 Mount"
-			(at 0 3.75 0)
+		(property "Value" "M2.5 mount"
+			(at 0 3.3 0)
 			(layer "F.Fab")
 			(effects
@@
 		(fp_circle
 			(center 0 0)
-			(end 2.8 0)
+			(end 2.35 0)
 			(stroke
 				(width 0.15)
@@
 		(fp_circle
 			(center 0 0)
-			(end 3.05 0)
+			(end 2.6 0)
 			(stroke
 				(width 0.05)
@@
 		(pad "1" thru_hole circle
 			(at 0 0)
-			(size 3.6 3.6)
-			(drill 3.2)
+			(size 3.1 3.1)
+			(drill 2.7)
 			(layers "*.Cu" "*.Mask")
 			(remove_unused_layers no)
@@
 		(pad "1" connect circle
 			(at 0 0)
-			(size 5.6 5.6)
+			(size 4.7 4.7)
 			(layers "F.Cu" "F.Mask")
 			(net "GND")
@@
 		)
 	)
-	(footprint "MountingHole:MountingHole_3.2mm_M3_DIN965"
+	(footprint "MountingHole:MountingHole_2.7mm_M2.5"
 		(layer "F.Cu")
 		(at 174 134)
-		(descr "Mounting Hole 3.2mm, M3, no annular, generated by kicad-footprint-generator mountinghole.py")
-		(tags "mountinghole M3 DIN965")
+		(descr "Mounting Hole 2.7mm, M2.5, no annular, generated by kicad-footprint-generator mountinghole.py")
+		(tags "mountinghole M2.5")
 		(property "Reference" "H2"
-			(at 0 -3.75 0)
+			(at 0 -3.65 0)
 			(layer "F.SilkS")
 			(effects
@@
 			)
 		)
-		(property "Value" "M3 mount"
-			(at 0 3.75 0)
+		(property "Value" "M2.5 mount"
+			(at 0 3.65 0)
 			(layer "F.Fab")
 			(effects
@@
 		(fp_circle
 			(center 0 0)
-			(end 2.8 0)
+			(end 2.7 0)
 			(stroke
 				(width 0.15)
@@
 		(fp_circle
 			(center 0 0)
-			(end 3.05 0)
+			(end 2.95 0)
 			(stroke
 				(width 0.05)
@@
 		(pad "" np_thru_hole circle
 			(at 0 0)
-			(size 3.2 3.2)
-			(drill 3.2)
+			(size 2.7 2.7)
+			(drill 2.7)
 			(layers "*.Cu" "*.Mask")
 		)
@@
 			)
 		)
-		(property "Value" "M3 mount"
+		(property "Value" "M2.5 mount"
 			(at 0 3.65 0)
 			(layer "F.Fab")
@@
 			)
 		)
-		(attr exclude_from_bom dnp)
+		(attr exclude_from_bom)
 		(duplicate_pad_numbers_are_jumpers no)
 		(fp_circle
@@
 		)
 	)
-	(footprint "MountingHole:MountingHole_3.2mm_M3_DIN965"
+	(footprint "MountingHole:MountingHole_2.7mm_M2.5"
 		(layer "F.Cu")
 		(at 82 134)
-		(descr "Mounting Hole 3.2mm, M3, no annular, generated by kicad-footprint-generator mountinghole.py")
-		(tags "mountinghole M3 DIN965")
+		(descr "Mounting Hole 2.7mm, M2.5, no annular, generated by kicad-footprint-generator mountinghole.py")
+		(tags "mountinghole M2.5")
 		(property "Reference" "H3"
-			(at 0 -3.75 0)
+			(at 0 -3.65 0)
 			(layer "F.SilkS")
 			(effects
@@
 			)
 		)
-		(property "Value" "M3 mount"
-			(at 0 3.75 0)
+		(property "Value" "M2.5 mount"
+			(at 0 3.65 0)
 			(layer "F.Fab")
 			(effects
@@
 		(fp_circle
 			(center 0 0)
-			(end 2.8 0)
+			(end 2.7 0)
 			(stroke
 				(width 0.15)
@@
 		(fp_circle
 			(center 0 0)
-			(end 3.05 0)
+			(end 2.95 0)
 			(stroke
 				(width 0.05)
@@
 		(pad "" np_thru_hole circle
 			(at 0 0)
-			(size 3.2 3.2)
-			(drill 3.2)
+			(size 2.7 2.7)
+			(drill 2.7)
 			(layers "*.Cu" "*.Mask")
 		)

Commit message: final touches, readme
Parts:
- removed R25, R28, R55: 0Ω, PCM_JLCPCB:R_0603
- added J10: Conn_01x02, Connector_PinHeader_2.54mm:PinHeader_1x02_P2.54mm_Vertical, F.Cu at (99.7, 109.0)
- added J11: Conn_01x02, Connector_PinHeader_2.54mm:PinHeader_1x02_P2.54mm_Vertical, F.Cu at (103.8, 111.3)
- added J8: Conn_01x02, Connector_JST:JST_XH_B2B-XH-A_1x02_P2.50mm_Vertical, F.Cu at (163.3, 133.7)
- added J9: Conn_01x02, Connector_PinHeader_2.54mm:PinHeader_1x02_P2.54mm_Vertical, F.Cu at (114.0, 110.6)
- turned R31 to 0 degrees
- turned R53 to 180 degrees
Connections:
- R31 pad 1: /OP_Gate_Out -> /OP_Gate_-
- R31 pad 2: /OP_Gate_- -> /OP_Gate_Out
- R53 pad 1: GND -> /OP_Gate_-
- R53 pad 2: /OP_Gate_- -> GND
- U5 pad 11: /Bus_switch/Chainbus.SCL -> /Bus_switch/Chainbus.SDA
- U5 pad 12: /Bus_switch/Chainbus.SDA -> /Bus_switch/Chainbus.SCL
Routing:
- net /Free: track 54.5 -> 77.6 mm, vias 2 -> 3
- net /PWM_P: track 85.3 -> 89.7 mm, vias 5 -> 7
- net +3V3: track 197.6 -> 200.2 mm
- net Net-(J10-Pin_2): track 2.91 -> 5.26 mm
- net /Mosfet_Feedback: track 45.6 -> 43.3 mm
- net /Bus_switch/Chainbus.SDA: track 77.8 -> 79.7 mm
- net /PWM_N: track 100.8 -> 102.5 mm
- net Net-(J9-Pin_2): track 3.27 -> 4.64 mm, vias 0 -> 1
- net /Sel_Output_amm: track 98.4 -> 99.5 mm
- net /Sel_Output_Volt: track 86.3 -> 87.3 mm
- net /Bus_switch/Chainbus.SCL: track 78.9 -> 78.2 mm
- net Net-(J11-Pin_2): track 3.29 -> 3.81 mm
- net GND: vias 88 -> 87
Other:
- board text added: "0V"
- board text added: "TX"

Commit message: fixed reserved pins
Connections:
- J1 pad 25: unconnected-(J1-Pin_25-Pad25) -> /Interboard_connector/R1
- J1 pad 27: unconnected-(J1-Pin_27-Pad27) -> /Interboard_connector/R2
- J2 pad 25: unconnected-(J2-Pin_25-Pad25) -> /Interboard_connector/R1
- J2 pad 27: unconnected-(J2-Pin_27-Pad27) -> /Interboard_connector/R2
Routing:
- net /Interboard_connector/R2: track 0.00 -> 2.56 mm, vias 0 -> 1
- net /Interboard_connector/R1: track 0.00 -> 2.13 mm, vias 0 -> 1
Changed lines of the file:
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@@
 			(size 3 1)
 			(layers "F.Cu" "F.Mask" "F.Paste")
-			(net "unconnected-(J2-Pin_25-Pad25)")
+			(net "/Interboard_connector/R1")
 			(pinfunction "Pin_25_25")
-			(pintype "passive+no_connect")
+			(pintype "passive")
 		)
 		(pad "26" smd rect
@@
 			(size 3 1)
 			(layers "F.Cu" "F.Mask" "F.Paste")
-			(net "unconnected-(J2-Pin_27-Pad27)")
+			(net "/Interboard_connector/R2")
 			(pinfunction "Pin_27_27")
-			(pintype "passive+no_connect")
+			(pintype "passive")
 		)
 		(pad "28" smd rect
@@
 			(size 3.15 1)
 			(layers "B.Cu" "B.Mask" "B.Paste")
-			(net "unconnected-(J1-Pin_25-Pad25)")
+			(net "/Interboard_connector/R1")
 			(pinfunction "Pin_25_25")
-			(pintype "passive+no_connect")
+			(pintype "passive")
 		)
 		(pad "26" smd rect
@@
 			(size 3.15 1)
 			(layers "B.Cu" "B.Mask" "B.Paste")
-			(net "unconnected-(J1-Pin_27-Pad27)")
+			(net "/Interboard_connector/R2")
 			(pinfunction "Pin_27_27")
-			(pintype "passive+no_connect")
+			(pintype "passive")
 		)
 		(pad "28" smd rect
@@
 		(net "/CH32V003/SWIO")
 	)
+	(segment
+		(start 139.43 93.038272)
+		(end 138.961728 93.038272)
+		(width 0.2)
+		(layer "F.Cu")
+		(net "/Interboard_connector/R1")
+	)
+	(segment
+		(start 138.961728 93.038272)
+		(end 138.4 93.6)
+		(width 0.2)
+		(layer "F.Cu")
+		(net "/Interboard_connector/R1")
+	)
+	(via
+		(at 138.4 93.6)
+		(size 0.5)
+		(drill 0.3)
+		(layers "F.Cu" "B.Cu")
+		(net "/Interboard_connector/R1")
+	)
+	(segment
+		(start 138.4 93.6)
+		(end 138.45 93.55)
+		(width 0.2)
+		(layer "B.Cu")
+		(net "/Interboard_connector/R1")
+	)
+	(segment
+		(start 138.45 93.55)
+		(end 139.25 93.55)
+		(width 0.2)
+		(layer "B.Cu")
+		(net "/Interboard_connector/R1")
+	)
+	(segment
+		(start 141.411728 93.038272)
+		(end 140.9 93.55)
+		(width 0.2)
+		(layer "F.Cu")
+		(net "/Interboard_connector/R2")
+	)
+	(segment
+		(start 141.97 93.038272)
+		(end 141.411728 93.038272)
+		(width 0.2)
+		(layer "F.Cu")
+		(net "/Interboard_connector/R2")
+	)
+	(via
+		(at 140.9 93.55)
+		(size 0.5)
+		(drill 0.3)
+		(layers "F.Cu" "B.Cu")
+		(net "/Interboard_connector/R2")
+	)
+	(segment
+		(start 141.423272 93.55)
+		(end 141.96 93.013272)
+		(width 0.2)
+		(layer "B.Cu")
+		(net "/Interboard_connector/R2")
+	)
+	(segment
+		(start 140.9 93.55)
+		(end 141.423272 93.55)
+		(width 0.2)
+		(layer "B.Cu")
+		(net "/Interboard_connector/R2")
+	)
 	(zone
